File: 0_assemb_full/stm32.kicad_sch (KiCad schematic)
At the start: 1 part, among them U24 STM32F091RCTx

Commit message: Additional changes
Parts:
- added C11, C12, C13, C15: 100n, symbol Device:C
- added C14, C16: 4.7u, symbol Device:C
- added C17: 10n, symbol Device:C
- added C18: 1u, symbol Device:C
- added C19: 0.1u, symbol Device:C
- added FB1: FerriteBead, symbol Device:FerriteBead
- added J4: Conn_01x02, symbol Connector_Generic:Conn_01x02
- added R58: 100K, symbol Device:R_US
Connections:
- net 3_3V: now reaches U24.1 (VBAT)
- net 3_3V: now also U24.19 (VDD), U24.32 (VDD), U24.48 (VDDIO2), U24.64 (VDD), C11.1, C12.1, C13.1, C14.1, C15.1, C16.1, FB1.1
- net GND: now reaches U24.12 (VSSA)
- net GND: now also U24.18 (VSS), U24.31 (VSS), U24.47 (VSS), U24.63 (VSS), C11.2, C12.2, C13.2, C14.2, C15.2, C16.2, C17.2, C18.2, C19.2, J4.2 (Pin_2), R58.1
- net VDDA: now reaches U24.13 (VDDA)
- net VDDA: now also C17.1, C18.1, FB1.2
- net Boot0: now reaches U24.60 (PF11)
- net Boot0: now also R58.2
- net NRST: now reaches U24.7 (NRST)
- net NRST: now also C19.1, J4.1 (Pin_1)
Other:
- note added: "600Ohm @ 100MHz .3 Ohm DCR, 500 mA"
- note added: "Boot0"
- note added: "Power Conditioning"
- note added: "Reset Jumper"

Commit message: Removed varistors, updated some STM32 connections
Parts:
- added J5: SPIConn_01x03, symbol Connector_Generic:Conn_01x03
Connections:
- net ADC_HP: now reaches U24.10 (PC2)
- net SPI_NSS: now reaches U24.33 (PB12)
- net SPI_NSS: now also J5.1 (Pin_1)
- net SPI_SCK: now reaches U24.34 (PB13)
- net SPI_SCK: now also J5.2 (Pin_2)
- net SPI_MOSI: now reaches U24.36 (PB15)
- net SPI_MOSI: now also J5.3 (Pin_3)
- net ADC_LP: now reaches U24.8 (PC0)
- net ADC_BP: now reaches U24.9 (PC1)
Other:
- moved on the sheet: R58
Changed lines of the file:
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@@
+    (stroke (width 0) (type default) (color 0 0 0 0))
+  )
+  (wire (pts (xy 152.4 134.62) (xy 166.37 134.62))
     (stroke (width 0) (type default) (color 0 0 0 0))
   )
@@
     (stroke (width 0) (type default) (color 0 0 0 0))
   )
-  (wire (pts (xy 58.42 92.71) (xy 58.42 91.44))
+  (wire (pts (xy 60.96 95.25) (xy 60.96 93.98))
     (stroke (width 0) (type default) (color 0 0 0 0))
   )
@@
     (stroke (width 0) (type default) (color 0 0 0 0))
   )
+  (wire (pts (xy 185.42 129.54) (xy 195.58 129.54))
+    (stroke (width 0) (type default) (color 0 0 0 0))
+  )
   (wire (pts (xy 30.48 93.98) (xy 30.48 95.25))
     (stroke (width 0) (type default) (color 0 0 0 0))
@@
     (stroke (width 0) (type default) (color 0 0 0 0))
   )
+  (wire (pts (xy 152.4 129.54) (xy 166.37 129.54))
+    (stroke (width 0) (type default) (color 0 0 0 0))
+  )
   (wire (pts (xy 59.69 74.93) (xy 59.69 73.66))
     (stroke (width 0) (type default) (color 0 0 0 0))
   )
+  (wire (pts (xy 105.41 101.6) (xy 119.38 101.6))
+    (stroke (width 0) (type default) (color 0 0 0 0))
+  )
   (wire (pts (xy 59.69 66.04) (xy 59.69 64.77))
     (stroke (width 0) (type default) (color 0 0 0 0))
   )
+  (wire (pts (xy 152.4 127) (xy 166.37 127))
+    (stroke (width 0) (type default) (color 0 0 0 0))
+  )
   (wire (pts (xy 52.07 30.48) (xy 59.69 30.48))
     (stroke (width 0) (type default) (color 0 0 0 0))
   )
-  (wire (pts (xy 58.42 91.44) (xy 59.69 91.44))
+  (wire (pts (xy 105.41 96.52) (xy 119.38 96.52))
+    (stroke (width 0) (type default) (color 0 0 0 0))
+  )
+  (wire (pts (xy 60.96 93.98) (xy 62.23 93.98))
+    (stroke (width 0) (type default) (color 0 0 0 0))
+  )
+  (wire (pts (xy 185.42 132.08) (xy 195.58 132.08))
     (stroke (width 0) (type default) (color 0 0 0 0))
   )
@@
     (stroke (width 0) (type default) (color 0 0 0 0))
   )
-  (wire (pts (xy 67.31 91.44) (xy 74.93 91.44))
+  (wire (pts (xy 69.85 93.98) (xy 77.47 93.98))
+    (stroke (width 0) (type default) (color 0 0 0 0))
+  )
+  (wire (pts (xy 105.41 99.06) (xy 119.38 99.06))
     (stroke (width 0) (type default) (color 0 0 0 0))
   )
@@
     (stroke (width 0) (type default) (color 0 0 0 0))
   )
+  (wire (pts (xy 185.42 127) (xy 195.58 127))
+    (stroke (width 0) (type default) (color 0 0 0 0))
+  )
   (wire (pts (xy 142.24 46.99) (xy 142.24 48.26))
     (stroke (width 0) (type default) (color 0 0 0 0))
@@
     (effects (font (size 1.27 1.27)) (justify left bottom))
   )
+  (label "SPI_MOSI" (at 185.42 132.08 0)
+    (effects (font (size 1.27 1.27)) (justify left bottom))
+  )
   (label "NRST" (at 15.24 91.44 0)
     (effects (font (size 1.27 1.27)) (justify left bottom))
   )
+  (label "SPI_MOSI" (at 166.37 134.62 180)
+    (effects (font (size 1.27 1.27)) (justify right bottom))
+  )
+  (label "SPI_SCK" (at 185.42 129.54 0)
+    (effects (font (size 1.27 1.27)) (justify left bottom))
+  )
   (label "VDD_In" (at 134.62 45.72 180)
     (effects (font (size 1.27 1.27)) (justify right bottom))
@@
     (effects (font (size 1.27 1.27)) (justify right bottom))
   )
-  (label "Boot0" (at 74.93 91.44 180)
+  (label "SPI_SCK" (at 166.37 129.54 180)
+    (effects (font (size 1.27 1.27)) (justify right bottom))
+  )
+  (label "Boot0" (at 77.47 93.98 180)
     (effects (font (size 1.27 1.27)) (justify right bottom))
   )
@@
     (effects (font (size 1.27 1.27)) (justify left bottom))
   )
+  (label "SPI_NSS" (at 185.42 127 0)
+    (effects (font (size 1.27 1.27)) (justify left bottom))
+  )
+  (label "SPI_NSS" (at 166.37 127 180)
+    (effects (font (size 1.27 1.27)) (justify right bottom))
+  )
   (label "VDD_In" (at 80.01 20.32 180)
     (effects (font (size 1.27 1.27)) (justify right bottom))
@@
     (effects (font (size 1.27 1.27)) (justify right bottom))
   )
+  (global_label "ADC_HP" (shape input) (at 105.41 101.6 180) (fields_autoplaced)
+    (effects (font (size 1.27 1.27)) (justify right))
+    (property "Intersheet References" "${INTERSHEET_REFS}" (id 0) (at 95.8002 101.5206 0)
+      (effects (font (size 1.27 1.27)) (justify right) hide)
+    )
+  )
+  (global_label "ADC_LP" (shape input) (at 105.41 96.52 180) (fields_autoplaced)
+    (effects (font (size 1.27 1.27)) (justify right))
+    (property "Intersheet References" "${INTERSHEET_REFS}" (id 0) (at 96.1026 96.4406 0)
+      (effects (font (size 1.27 1.27)) (justify right) hide)
+    )
+  )
   (global_label "3_3V" (shape input) (at 25.4 64.77 180) (fields_autoplaced)
     (effects (font (size 1.27 1.27)) (justify right))
@@
     )
   )
+  (global_label "ADC_BP" (shape input) (at 105.41 99.06 180) (fields_autoplaced)
+    (effects (font (size 1.27 1.27)) (justify right))
+    (property "Intersheet References" "${INTERSHEET_REFS}" (id 0) (at 95.8607 98.9806 0)
+      (effects (font (size 1.27 1.27)) (justify right) hide)
+    )
+  )
   (global_label "3_3V" (shape input) (at 25.4 40.64 180) (fields_autoplaced)
     (effects (font (size 1.27 1.27)) (justify right))
@@
     (pin "2")
   )
-  (symbol (lib_id "Device:R_US") (at 63.5 91.44 90) (unit 1)
-    (in_bom yes) (on_board yes) (fields_autoplaced)
-    (property "Reference" "R58" (id 0) (at 63.5 85.09 90))
-    (property "Value" "100K" (id 1) (at 63.5 87.63 90))
-    (property "Footprint" "" (id 2) (at 63.754 90.424 90)
-      (effects (font (size 1.27 1.27)) hide)
-    )
-    (property "Datasheet" "~" (id 3) (at 63.5 91.44 0)
+  (symbol (lib_id "Connector_Generic:Conn_01x03") (at 200.66 129.54 0) (unit 1)
+    (in_bom yes) (on_board yes) (fields_autoplaced)
+    (property "Reference" "J5" (id 0) (at 203.2 128.2699 0)
+      (effects (font (size 1.27 1.27)) (justify left))
+    )
+    (property "Value" "SPIConn_01x03" (id 1) (at 203.2 130.8099 0)
+      (effects (font (size 1.27 1.27)) (justify left))
+    )
+    (property "Footprint" "" (id 2) (at 200.66 129.54 0)
+      (effects (font (size 1.27 1.27)) hide)
+    )
+    (property "Datasheet" "~" (id 3) (at 200.66 129.54 0)
+      (effects (font (size 1.27 1.27)) hide)
+    )
+    (pin "1")
+    (pin "2")
+    (pin "3")
+  )
+  (symbol (lib_id "Device:R_US") (at 66.04 93.98 90) (unit 1)
+    (in_bom yes) (on_board yes) (fields_autoplaced)
+    (property "Reference" "R58" (id 0) (at 66.04 87.63 90))
+    (property "Value" "100K" (id 1) (at 66.04 90.17 90))
+    (property "Footprint" "" (id 2) (at 66.294 92.964 90)
+      (effects (font (size 1.27 1.27)) hide)
+    )
+    (property "Datasheet" "~" (id 3) (at 66.04 93.98 0)
       (effects (font (size 1.27 1.27)) hide)
     )
@@
     (pin "2")
   )
-  (symbol (lib_id "power:GND") (at 58.42 92.71 0) (unit 1)
-    (in_bom yes) (on_board yes) (fields_autoplaced)
-    (property "Reference" "#PWR030" (id 0) (at 58.42 99.06 0)
-      (effects (font (size 1.27 1.27)) hide)
-    )
-    (property "Value" "GND" (id 1) (at 58.42 97.79 0)
-      (effects (font (size 1.27 1.27)) hide)
-    )
-    (property "Footprint" "" (id 2) (at 58.42 92.71 0)
-      (effects (font (size 1.27 1.27)) hide)
-    )
-    (property "Datasheet" "" (id 3) (at 58.42 92.71 0)
-      (effects (font (size 1.27 1.27)) hide)
-    )
+  (symbol (lib_id "power:GND") (at 60.96 95.25 0) (unit 1)
+    (in_bom yes) (on_board yes) (fields_autoplaced)
+    (property "Reference" "#PWR030" (id 0) (at 60.96 101.6 0)
+      (effects (font (size 1.27 1.27)) hide)
+    )
+    (property "Value" "GND" (id 1) (at 60.96 100.33 0)
+      (effects (font (size 1.27 1.27)) hide)
+    )
+    (property "Footprint" "" (id 2) (at 60.96 95.25 0)
+      (effects (font (size 1.27 1.27)) hide)
+    )
+    (property "Datasheet" "" (id 3) (at 60.96 95.25 0)
+      (effects (font (size 1.27 1.27)) hide)
+    )

Commit message: Bandpass filter all set now!
Parts:
- renumbered C11 to C13, C12 to C14, C13 to C15, C14 to C16, C15 to C17, C16 to C18, C17 to C19, C18 to C20, C19 to C21, R58 to R62, U24 to U25
Changed lines of the file:
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@@
   (symbol (lib_id "Device:C") (at 31.75 45.72 0) (unit 1)
     (in_bom yes) (on_board yes) (fields_autoplaced)
-    (property "Reference" "C15" (id 0) (at 35.56 44.4499 0)
+    (property "Reference" "C17" (id 0) (at 35.56 44.4499 0)
       (effects (font (size 1.27 1.27)) (justify left))
     )
@@
   (symbol (lib_id "Device:R_US") (at 66.04 93.98 90) (unit 1)
     (in_bom yes) (on_board yes) (fields_autoplaced)
-    (property "Reference" "R58" (id 0) (at 66.04 87.63 90))
+    (property "Reference" "R62" (id 0) (at 66.04 87.63 90))
     (property "Value" "100K" (id 1) (at 66.04 90.17 90))
     (property "Footprint" "" (id 2) (at 66.294 92.964 90)
@@
   (symbol (lib_id "Device:C") (at 31.75 25.4 0) (unit 1)
     (in_bom yes) (on_board yes) (fields_autoplaced)
-    (property "Reference" "C11" (id 0) (at 35.56 24.1299 0)
+    (property "Reference" "C13" (id 0) (at 35.56 24.1299 0)
       (effects (font (size 1.27 1.27)) (justify left))
     )
@@
   (symbol (lib_id "Device:C") (at 59.69 25.4 0) (unit 1)
     (in_bom yes) (on_board yes) (fields_autoplaced)
-    (property "Reference" "C13" (id 0) (at 63.5 24.1299 0)
+    (property "Reference" "C15" (id 0) (at 63.5 24.1299 0)
       (effects (font (size 1.27 1.27)) (justify left))
     )
@@
   (symbol (lib_id "power:GND") (at 30.48 95.25 0) (unit 1)
     (in_bom yes) (on_board yes) (fields_autoplaced)
-    (property "Reference" "#PWR031" (id 0) (at 30.48 101.6 0)
+    (property "Reference" "#PWR030" (id 0) (at 30.48 101.6 0)
       (effects (font (size 1.27 1.27)) hide)
     )
@@
   (symbol (lib_id "Device:C") (at 45.72 45.72 0) (unit 1)
     (in_bom yes) (on_board yes) (fields_autoplaced)
-    (property "Reference" "C16" (id 0) (at 49.53 44.4499 0)
+    (property "Reference" "C18" (id 0) (at 49.53 44.4499 0)
       (effects (font (size 1.27 1.27)) (justify left))
     )
@@
   (symbol (lib_id "Device:C") (at 45.72 69.85 0) (unit 1)
     (in_bom yes) (on_board yes) (fields_autoplaced)
-    (property "Reference" "C17" (id 0) (at 49.53 68.5799 0)
+    (property "Reference" "C19" (id 0) (at 49.53 68.5799 0)
       (effects (font (size 1.27 1.27)) (justify left))
     )
@@
   (symbol (lib_id "Device:C") (at 73.66 25.4 0) (unit 1)
     (in_bom yes) (on_board yes) (fields_autoplaced)
-    (property "Reference" "C14" (id 0) (at 77.47 24.1299 0)
+    (property "Reference" "C16" (id 0) (at 77.47 24.1299 0)
       (effects (font (size 1.27 1.27)) (justify left))
     )
@@
   (symbol (lib_id "Device:C") (at 20.32 95.25 0) (unit 1)
     (in_bom yes) (on_board yes) (fields_autoplaced)
-    (property "Reference" "C19" (id 0) (at 24.13 93.9799 0)
+    (property "Reference" "C21" (id 0) (at 24.13 93.9799 0)
       (effects (font (size 1.27 1.27)) (justify left))
     )
@@
   (symbol (lib_id "power:GND") (at 60.96 95.25 0) (unit 1)
     (in_bom yes) (on_board yes) (fields_autoplaced)
-    (property "Reference" "#PWR030" (id 0) (at 60.96 101.6 0)
+    (property "Reference" "#PWR031" (id 0) (at 60.96 101.6 0)
       (effects (font (size 1.27 1.27)) hide)
     )
@@
   (symbol (lib_id "MCU_ST_STM32F0:STM32F091RCTx") (at 137.16 93.98 0) (unit 1)
     (in_bom yes) (on_board yes) (fields_autoplaced)
-    (property "Reference" "U24" (id 0) (at 141.7194 139.7 0)
+    (property "Reference" "U25" (id 0) (at 141.7194 139.7 0)
       (effects (font (size 1.27 1.27)) (justify left))
     )
@@
   (symbol (lib_id "Device:C") (at 59.69 69.85 0) (unit 1)
     (in_bom yes) (on_board yes) (fields_autoplaced)
-    (property "Reference" "C18" (id 0) (at 63.5 68.5799 0)
+    (property "Reference" "C20" (id 0) (at 63.5 68.5799 0)
       (effects (font (size 1.27 1.27)) (justify left))
     )
@@
   (symbol (lib_id "Device:C") (at 45.72 25.4 0) (unit 1)
     (in_bom yes) (on_board yes) (fields_autoplaced)
-    (property "Reference" "C12" (id 0) (at 49.53 24.1299 0)
-      (effects (font (size 1.27 1.27)) (justify left))
-    )
+    (property "Reference" "C14" (id 0) (at 49.53 24.1299 0)
+      (effects (font (size 1.27 1.27)) (justify left))
+    )

Commit message: A bunch of changes to the schematics
Parts:
- removed C13, C17: 100n, symbol Device:C
- removed C16, C18: 4.7u, symbol Device:C
- removed C19: 10n, symbol Device:C
- removed C20: 1u, symbol Device:C
- added C? (x2): 4.7u, symbol Device:C
- added C?: 10n, symbol Device:C
- added C? (x2): 100n, symbol Device:C
- added C?: 1u, symbol Device:C
- added R?: 100K, symbol Device:R_US
Connections:
- net 3_3V: now also C?.1, C?.1, C?.1, C?.1, R?.2
- net GND: now also C?.2, C?.2, C?.2, C?.2, C?.2, C?.2
- net NRST: now also R?.1
- net VDDA: now also C?.1, C?.1
- net SERVO4: now reaches U25.15 (PA1)
- net SERVO0: now reaches U25.41 (PA8)
- net SERVO1: now reaches U25.42 (PA9)
- net SERVO2: now reaches U25.43 (PA10)
- net SERVO3: now reaches U25.44 (PA11)
