File: 0_assemb_full/assemb_full.kicad_sch (KiCad schematic)
At the start: 18 parts, among them J1 BarrelJack, J11 OutToRPi, J2 Conn_02x06, J3 AudioJack3, J4 Servo0Conn_01x03, J5 Servo1Conn_01x03, J6 Servo2Conn_01x03, J7 Servo3Conn_01x03, J8 Servo4Conn_01x03, U1 LM2902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

Commit message: Pre-STM32 portion rework
Parts:
- H1, H2, H3, H4: footprint MountingHole:MountingHole_6.4mm_M6 -> MountingHole:MountingHole_3.2mm_M3
Changed lines of the file:
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@@
       (effects (font (size 1.27 1.27)) (justify left))
     )
-    (property "Footprint" "MountingHole:MountingHole_6.4mm_M6" (id 2) (at 97.79 154.94 0)
+    (property "Footprint" "MountingHole:MountingHole_3.2mm_M3" (id 2) (at 97.79 154.94 0)
       (effects (font (size 1.27 1.27)) hide)
     )
@@
       (effects (font (size 1.27 1.27)) (justify left))
     )
-    (property "Footprint" "MountingHole:MountingHole_6.4mm_M6" (id 2) (at 77.47 154.94 0)
+    (property "Footprint" "MountingHole:MountingHole_3.2mm_M3" (id 2) (at 77.47 154.94 0)
       (effects (font (size 1.27 1.27)) hide)
     )
@@
       (effects (font (size 1.27 1.27)) (justify left))
     )
-    (property "Footprint" "MountingHole:MountingHole_6.4mm_M6" (id 2) (at 77.47 162.56 0)
+    (property "Footprint" "MountingHole:MountingHole_3.2mm_M3" (id 2) (at 77.47 162.56 0)
       (effects (font (size 1.27 1.27)) hide)
     )
@@
       (effects (font (size 1.27 1.27)) (justify left))
     )
-    (property "Footprint" "MountingHole:MountingHole_6.4mm_M6" (id 2) (at 97.79 162.56 0)
+    (property "Footprint" "MountingHole:MountingHole_3.2mm_M3" (id 2) (at 97.79 162.56 0)
       (effects (font (size 1.27 1.27)) hide)
     )
@@
       (reference "#PWR023") (unit 1) (value "GND") (footprint "")
     )
+    (path "/4d0bd211-4794-4141-8b4c-fc5ed36fe38a/72e1a72a-73f3-4e77-9cc1-64502cad8971"
+      (reference "#PWR024") (unit 1) (value "GND") (footprint "")
+    )
     (path "/4d0bd211-4794-4141-8b4c-fc5ed36fe38a/dffc0aac-0aa8-46f6-bf11-363286084e9a"
       (reference "#PWR025") (unit 1) (value "GND") (footprint "")
@@
       (reference "#PWR044") (unit 1) (value "GND") (footprint "")
     )
+    (path "/4d0bd211-4794-4141-8b4c-fc5ed36fe38a/006e9ca3-93e1-436f-bcb0-b6de89c35cff"
+      (reference "#PWR045") (unit 1) (value "GND") (footprint "")
+    )
     (path "/701dbde4-06b5-452b-9745-23728d983406"
       (reference "#PWR0101") (unit 1) (value "GND") (footprint "")
@@
       (reference "C49") (unit 1) (value "1000p") (footprint "Capacitor_SMD:C_0805_2012Metric_Pad1.18x1.45mm_HandSolder")
     )
+    (path "/4d0bd211-4794-4141-8b4c-fc5ed36fe38a/fc4a95b0-c222-4472-8389-28a3852fca31"
+      (reference "C50") (unit 1) (value "0.1u") (footprint "Capacitor_SMD:C_0805_2012Metric_Pad1.18x1.45mm_HandSolder")
+    )
     (path "/4d0bd211-4794-4141-8b4c-fc5ed36fe38a/822db18f-48d7-4f8b-90ac-b1d8ccd6b4ed"
       (reference "FB1") (unit 1) (value "FerriteBead") (footprint "Resistor_SMD:R_0805_2012Metric_Pad1.20x1.40mm_HandSolder")
@@
     )
     (path "/5cd393c2-fe36-4948-8074-481fc7601eb3"
-      (reference "H1") (unit 1) (value "MountingHole") (footprint "MountingHole:MountingHole_6.4mm_M6")
+      (reference "H1") (unit 1) (value "MountingHole") (footprint "MountingHole:MountingHole_3.2mm_M3")
     )
     (path "/553fbf29-cee2-4c40-b73f-a88188719d8f"
-      (reference "H2") (unit 1) (value "MountingHole") (footprint "MountingHole:MountingHole_6.4mm_M6")
+      (reference "H2") (unit 1) (value "MountingHole") (footprint "MountingHole:MountingHole_3.2mm_M3")
     )
     (path "/79a8d5eb-9c1a-4b82-9a43-f5f942096787"
-      (reference "H3") (unit 1) (value "MountingHole") (footprint "MountingHole:MountingHole_6.4mm_M6")
+      (reference "H3") (unit 1) (value "MountingHole") (footprint "MountingHole:MountingHole_3.2mm_M3")
     )
     (path "/d0417bfa-517d-41a0-a9a3-7574aae19384"
-      (reference "H4") (unit 1) (value "MountingHole") (footprint "MountingHole:MountingHole_6.4mm_M6")
+      (reference "H4") (unit 1) (value "MountingHole") (footprint "MountingHole:MountingHole_3.2mm_M3")
     )
     (path "/3e1ccb16-5496-4985-9aa9-d268c89cac5f"
@@
       (reference "U6") (unit 1) (value "TPA3138D2PWP") (footprint "Specifics:IC_TPS61196PWPRQ1")
     )
-  )
+    (path "/4d0bd211-4794-4141-8b4c-fc5ed36fe38a/dceda6e1-ad66-458a-ad2b-e62ed900e637"
+      (reference "U7") (unit 1) (value "MAX7375AXR805") (footprint "Package_TO_SOT_SMD:SOT-323_SC-70")
+    )
+  )

Commit message: Additional changes
Parts:
- C2: footprint Capacitor_THT:CP_Radial_D5.0mm_P2.00mm -> Capacitor_SMD:C_0805_2012Metric_Pad1.18x1.45mm_HandSolder
Changed lines of the file:
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@@
       (effects (font (size 1.27 1.27)) (justify left))
     )
-    (property "Footprint" "Capacitor_THT:CP_Radial_D5.0mm_P2.00mm" (id 2) (at 271.4752 72.39 0)
+    (property "Footprint" "Capacitor_SMD:C_0805_2012Metric_Pad1.18x1.45mm_HandSolder" (id 2) (at 271.4752 72.39 0)
       (effects (font (size 1.27 1.27)) hide)
     )
@@
     )
     (path "/6919c82c-5f1b-4169-8726-0ddf4f7a4d94"
-      (reference "C2") (unit 1) (value "10u") (footprint "Capacitor_THT:CP_Radial_D5.0mm_P2.00mm")
+      (reference "C2") (unit 1) (value "10u") (footprint "Capacitor_SMD:C_0805_2012Metric_Pad1.18x1.45mm_HandSolder")
     )
     (path "/27872fd8-6da5-4d41-bede-b1346c5a5ef3/ff4868b7-42c4-4637-8982-51f4c00414a6"
@@
     )
     (path "/4d0bd211-4794-4141-8b4c-fc5ed36fe38a/1bc0581a-1781-4e1b-8e60-5ca2d2b46f8a"
-      (reference "C13") (unit 1) (value "4.7u") (footprint "Capacitor_THT:CP_Radial_D5.0mm_P2.50mm")
+      (reference "C13") (unit 1) (value "4.7u") (footprint "Capacitor_SMD:C_0805_2012Metric_Pad1.18x1.45mm_HandSolder")
     )
     (path "/4d0bd211-4794-4141-8b4c-fc5ed36fe38a/fde15cd2-2cda-4c44-8d33-7c62ae44fe62"
@@
     )
     (path "/4d0bd211-4794-4141-8b4c-fc5ed36fe38a/f0546058-1d70-4ab5-a849-da358d11c444"
-      (reference "C17") (unit 1) (value "4.7u") (footprint "Capacitor_THT:CP_Radial_D5.0mm_P2.50mm")
+      (reference "C17") (unit 1) (value "4.7u") (footprint "Capacitor_SMD:C_0805_2012Metric_Pad1.18x1.45mm_HandSolder")
     )
     (path "/4d0bd211-4794-4141-8b4c-fc5ed36fe38a/9b233c35-f714-4c11-8775-60d1b489435f"
@@
     )
     (path "/4d0bd211-4794-4141-8b4c-fc5ed36fe38a/9c7263a0-5d7d-4638-a93a-5cc2c57952fb"
-      (reference "C19") (unit 1) (value "1u") (footprint "Capacitor_THT:CP_Radial_D5.0mm_P2.50mm")
+      (reference "C19") (unit 1) (value "1u") (footprint "Capacitor_SMD:C_0805_2012Metric_Pad1.18x1.45mm_HandSolder")
     )
     (path "/4d0bd211-4794-4141-8b4c-fc5ed36fe38a/74b03540-aa5e-4f88-abef-5190ace5f287"
@@
     )
     (path "/8dc894f1-9f5e-4081-ad24-6e5a5b7c14be/feba6847-64fc-402d-a2f6-ecfd5137a222"
-      (reference "C22") (unit 1) (value "1u") (footprint "Capacitor_THT:CP_Radial_D5.0mm_P2.50mm")
+      (reference "C22") (unit 1) (value "1u") (footprint "Capacitor_SMD:C_0805_2012Metric_Pad1.18x1.45mm_HandSolder")
     )
     (path "/8dc894f1-9f5e-4081-ad24-6e5a5b7c14be/fbb32664-578a-4db8-9d16-798563cdad4a"
-      (reference "C23") (unit 1) (value "1u") (footprint "Capacitor_THT:CP_Radial_D5.0mm_P2.50mm")
+      (reference "C23") (unit 1) (value "1u") (footprint "Capacitor_SMD:C_0805_2012Metric_Pad1.18x1.45mm_HandSolder")
     )
     (path "/8dc894f1-9f5e-4081-ad24-6e5a5b7c14be/1e1f34fd-5232-4cc7-ae2a-2de43ea493d4"
@@
     )
     (path "/8dc894f1-9f5e-4081-ad24-6e5a5b7c14be/5182e8ef-314e-48bf-997e-6ef46ec81aea"
-      (reference "C36") (unit 1) (value "1u") (footprint "Capacitor_THT:CP_Radial_D5.0mm_P2.50mm")
+      (reference "C36") (unit 1) (value "1u") (footprint "Capacitor_SMD:C_0805_2012Metric_Pad1.18x1.45mm_HandSolder")
     )
     (path "/8dc894f1-9f5e-4081-ad24-6e5a5b7c14be/84d7b5dc-cd48-4644-b842-c1b9ed0fb115"
-      (reference "C37") (unit 1) (value "1u") (footprint "Capacitor_THT:CP_Radial_D5.0mm_P2.50mm")
+      (reference "C37") (unit 1) (value "1u") (footprint "Capacitor_SMD:C_0805_2012Metric_Pad1.18x1.45mm_HandSolder")
     )
     (path "/8dc894f1-9f5e-4081-ad24-6e5a5b7c14be/552d0ae9-ab2f-4877-9380-e22ac2f5c271"
-      (reference "C38") (unit 1) (value "1u") (footprint "Capacitor_THT:CP_Radial_D5.0mm_P2.50mm")
+      (reference "C38") (unit 1) (value "1u") (footprint "Capacitor_SMD:C_0805_2012Metric_Pad1.18x1.45mm_HandSolder")
     )
     (path "/8dc894f1-9f5e-4081-ad24-6e5a5b7c14be/d546fde7-3607-4ea4-9e0e-dbf7c1255e90"
-      (reference "C39") (unit 1) (value "1u") (footprint "Capacitor_THT:CP_Radial_D5.0mm_P2.50mm")
+      (reference "C39") (unit 1) (value "1u") (footprint "Capacitor_SMD:C_0805_2012Metric_Pad1.18x1.45mm_HandSolder")
     )
     (path "/8dc894f1-9f5e-4081-ad24-6e5a5b7c14be/7c7883da-c220-4922-89c2-f5de5ef1b95e"

Commit message: Some filter adjustments
Parts:
- added C51: 100n, Capacitor_SMD:C_0805_2012Metric_Pad1.18x1.45mm_HandSolder, symbol Device:C_Small
- J2: footprint Connector_PinSocket_2.54mm:PinSocket_2x06_P2.54mm_Vertical -> Connector_PinHeader_2.54mm:PinHeader_2x02_P2.54mm_Vertical; symbol Connector_Generic:Conn_02x06_Odd_Even -> Connector_Generic:Conn_02x02_Odd_Even
- J4, J5, J6, J7, J8: footprint Connector_PinSocket_2.54mm:PinSocket_1x03_P2.54mm_Vertical -> Connector_PinHeader_2.54mm:PinHeader_1x03_P2.54mm_Vertical
Connections:
- net 12V: now also J2.1 (Pin_1); no longer J2.7 (Pin_7), J2.8 (Pin_8)
- net 5V: now also J2.3 (Pin_3), C51.1; no longer J2.1 (Pin_1), J2.2 (Pin_2)
- net GND: now also J2.2 (Pin_2), C51.2; no longer J2.3 (Pin_3), J2.5 (Pin_5), J2.6 (Pin_6)
- removed net 12VRP: J2.10 (Pin_10), J2.9 (Pin_9)
- removed net ENB: J2.11 (Pin_11)
- removed net PGB: J2.12 (Pin_12)

Commit message: Active Filters layout added
Other:
- title: (none) -> Power and Board I/O
Changed lines of the file:
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@@
 (kicad_sch (version 20211123) (generator eeschema)
   (paper "A4")
+  (title_block
+    (title "Power and Board I/O")
+  )
   (junction (at 252.73 45.72) (diameter 0) (color 0 0 0 0)
   )
@@
       (reference "#PWR013") (unit 1) (value "GND") (footprint "")
     )
-    (path "/27872fd8-6da5-4d41-bede-b1346c5a5ef3/f65b347d-1906-41a8-a443-040d2c14d2f3"
-      (reference "#PWR014") (unit 1) (value "GND") (footprint "")
-    )
     (path "/016209f3-6b0c-4be6-bf7f-4e52cc050e04/00c51497-9409-4520-8a70-92b48d98715b"
       (reference "#PWR015") (unit 1) (value "GND") (footprint "")
@@
     )
     (path "/8dc894f1-9f5e-4081-ad24-6e5a5b7c14be/2cdf5a20-566d-409f-92cf-c066a4af248f"
-      (reference "LS1") (unit 1) (value "8 ohms") (footprint "Connector_Wire:SolderWire-2.5sqmm_1x02_P7.2mm_D2.4mm_OD3.6mm")
+      (reference "LS1") (unit 1) (value "8 ohms") (footprint "Connector_Wire:SolderWire-2sqmm_1x02_P7.8mm_D2mm_OD3.9mm")
     )
     (path "/8dc894f1-9f5e-4081-ad24-6e5a5b7c14be/41db7f69-e5f0-4766-b41d-b0ac805900db"
-      (reference "LS2") (unit 1) (value "8 ohms") (footprint "Connector_Wire:SolderWire-2.5sqmm_1x02_P7.2mm_D2.4mm_OD3.6mm")
+      (reference "LS2") (unit 1) (value "8 ohms") (footprint "Connector_Wire:SolderWire-2sqmm_1x02_P7.8mm_D2mm_OD3.9mm")
     )
     (path "/8dc894f1-9f5e-4081-ad24-6e5a5b7c14be/b519694f-a9a7-4906-a169-735fae136041"
-      (reference "LS3") (unit 1) (value "8 ohms") (footprint "Connector_Wire:SolderWire-2.5sqmm_1x02_P7.2mm_D2.4mm_OD3.6mm")
+      (reference "LS3") (unit 1) (value "8 ohms") (footprint "Connector_Wire:SolderWire-2sqmm_1x02_P7.8mm_D2mm_OD3.9mm")
     )
     (path "/8dc894f1-9f5e-4081-ad24-6e5a5b7c14be/19bbda56-812e-467b-b4c1-9d41b601a6be"
-      (reference "LS4") (unit 1) (value "8 ohms") (footprint "Connector_Wire:SolderWire-2.5sqmm_1x02_P7.2mm_D2.4mm_OD3.6mm")
+      (reference "LS4") (unit 1) (value "8 ohms") (footprint "Connector_Wire:SolderWire-2sqmm_1x02_P7.8mm_D2mm_OD3.9mm")
     )
     (path "/27872fd8-6da5-4d41-bede-b1346c5a5ef3/5a4d8b69-7354-4d43-b6c0-a8ca9be8d8c7"
@@
       (reference "R11") (unit 1) (value "120") (footprint "Resistor_SMD:R_0805_2012Metric_Pad1.20x1.40mm_HandSolder")
     )
-    (path "/27872fd8-6da5-4d41-bede-b1346c5a5ef3/7411e74d-2ac9-4356-ae29-fd8399af3f31"
-      (reference "R12") (unit 1) (value "220") (footprint "Resistor_SMD:R_0805_2012Metric_Pad1.20x1.40mm_HandSolder")
-    )
-    (path "/27872fd8-6da5-4d41-bede-b1346c5a5ef3/536601fe-b1bf-4eca-9e23-e525e8086e7f"
-      (reference "R13") (unit 1) (value "220") (footprint "Resistor_SMD:R_0805_2012Metric_Pad1.20x1.40mm_HandSolder")
-    )
-    (path "/27872fd8-6da5-4d41-bede-b1346c5a5ef3/3245bbfe-7533-4f4e-8751-65166ad30d33"
-      (reference "R14") (unit 1) (value "220") (footprint "Resistor_SMD:R_0805_2012Metric_Pad1.20x1.40mm_HandSolder")
-    )
-    (path "/27872fd8-6da5-4d41-bede-b1346c5a5ef3/28b732bb-c589-40eb-b5c8-75949f6459e6"
-      (reference "R15") (unit 1) (value "220") (footprint "Resistor_SMD:R_0805_2012Metric_Pad1.20x1.40mm_HandSolder")
-    )
-    (path "/27872fd8-6da5-4d41-bede-b1346c5a5ef3/317bb91a-dacc-486d-8820-d84d8e4ef061"
-      (reference "R16") (unit 1) (value "220") (footprint "Resistor_SMD:R_0805_2012Metric_Pad1.20x1.40mm_HandSolder")
-    )
-    (path "/27872fd8-6da5-4d41-bede-b1346c5a5ef3/3612d0f6-a6f5-4ef7-8d12-2c00f1b34391"
-      (reference "R17") (unit 1) (value "220") (footprint "Resistor_SMD:R_0805_2012Metric_Pad1.20x1.40mm_HandSolder")
-    )
-    (path "/27872fd8-6da5-4d41-bede-b1346c5a5ef3/ebdfd93c-5c75-4510-bdc8-d4ca58791039"
-      (reference "R18") (unit 1) (value "220") (footprint "Resistor_SMD:R_0805_2012Metric_Pad1.20x1.40mm_HandSolder")
-    )
-    (path "/27872fd8-6da5-4d41-bede-b1346c5a5ef3/a425dd13-2c9a-4d72-a2f2-746e6c9237be"
-      (reference "R19") (unit 1) (value "220") (footprint "Resistor_SMD:R_0805_2012Metric_Pad1.20x1.40mm_HandSolder")
-    )
     (path "/016209f3-6b0c-4be6-bf7f-4e52cc050e04/6322e136-6565-4534-9cec-e553b466d6c3"

Commit message: Final adjustments
Parts:
- added J12: LEDConn_01x05, Connector_PinHeader_2.54mm:PinHeader_1x05_P2.54mm_Vertical, symbol Connector_Generic:Conn_01x05
Connections:
- net 5V: now also J12.5 (Pin_5)
- net GND: now also J12.4 (Pin_4)
- new net ADC_BP: J12.2 (Pin_2)
- new net ADC_HP: J12.1 (Pin_1)
- new net ADC_LP: J12.3 (Pin_3)
Changed lines of the file:
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@@
+    (stroke (width 0) (type default) (color 0 0 0 0))
+  )
+  (wire (pts (xy 68.58 191.77) (xy 59.69 191.77))
     (stroke (width 0) (type default) (color 0 0 0 0))
   )
@@
     (stroke (width 0) (type default) (color 0 0 0 0))
   )
+  (wire (pts (xy 59.69 191.77) (xy 59.69 193.04))
+    (stroke (width 0) (type default) (color 0 0 0 0))
+  )
   (wire (pts (xy 257.81 74.93) (xy 270.51 74.93))
     (stroke (width 0) (type default) (color 0 0 0 0))
@@
   )
   (wire (pts (xy 243.84 20.32) (xy 242.57 20.32))
+    (stroke (width 0) (type default) (color 0 0 0 0))
+  )
+  (wire (pts (xy 67.31 194.31) (xy 68.58 194.31))
     (stroke (width 0) (type default) (color 0 0 0 0))
   )
@@
   (text "Buck Connections" (at 236.22 53.34 0)
     (effects (font (size 1.27 1.27)) (justify left bottom))
+  )
+  (global_label "ADC_BP" (shape input) (at 68.58 186.69 180) (fields_autoplaced)
+    (effects (font (size 1.27 1.27)) (justify right))
+    (property "Intersheet References" "${INTERSHEET_REFS}" (id 0) (at 59.0307 186.6106 0)
+      (effects (font (size 1.27 1.27)) (justify right) hide)
+    )
+  )
+  (global_label "5V" (shape input) (at 67.31 194.31 180) (fields_autoplaced)
+    (effects (font (size 1.27 1.27)) (justify right))
+    (property "Intersheet References" "${INTERSHEET_REFS}" (id 0) (at 62.5988 194.2306 0)
+      (effects (font (size 1.27 1.27)) (justify right) hide)
+    )
   )
   (global_label "5V" (shape input) (at 21.59 179.07 180) (fields_autoplaced)
@@
     )
   )
+  (global_label "ADC_LP" (shape input) (at 68.58 189.23 180) (fields_autoplaced)
+    (effects (font (size 1.27 1.27)) (justify right))
+    (property "Intersheet References" "${INTERSHEET_REFS}" (id 0) (at 59.2726 189.1506 0)
+      (effects (font (size 1.27 1.27)) (justify right) hide)
+    )
+  )
   (global_label "5V" (shape input) (at 21.59 167.64 180) (fields_autoplaced)
     (effects (font (size 1.27 1.27)) (justify right))
@@
     (effects (font (size 1.27 1.27)) (justify right))
     (property "Intersheet References" "${INTERSHEET_REFS}" (id 0) (at 16.8788 156.1306 0)
+      (effects (font (size 1.27 1.27)) (justify right) hide)
+    )
+  )
+  (global_label "ADC_HP" (shape input) (at 68.58 184.15 180) (fields_autoplaced)
+    (effects (font (size 1.27 1.27)) (justify right))
+    (property "Intersheet References" "${INTERSHEET_REFS}" (id 0) (at 58.9702 184.0706 0)
       (effects (font (size 1.27 1.27)) (justify right) hide)
     )
@@
     (pin "3")
   )
+  (symbol (lib_id "Connector_Generic:Conn_01x05") (at 73.66 189.23 0) (unit 1)
+    (in_bom yes) (on_board yes) (fields_autoplaced)
+    (property "Reference" "J12" (id 0) (at 76.2 187.9599 0)
+      (effects (font (size 1.27 1.27)) (justify left))
+    )
+    (property "Value" "LEDConn_01x05" (id 1) (at 76.2 190.4999 0)
+      (effects (font (size 1.27 1.27)) (justify left))
+    )
+    (property "Footprint" "Connector_PinHeader_2.54mm:PinHeader_1x05_P2.54mm_Vertical" (id 2) (at 73.66 189.23 0)
+      (effects (font (size 1.27 1.27)) hide)
+    )
+    (property "Datasheet" "~" (id 3) (at 73.66 189.23 0)
+      (effects (font (size 1.27 1.27)) hide)
+    )
+    (pin "1")
+    (pin "2")
+    (pin "3")
+    (pin "4")
+    (pin "5")
+  )
   (symbol (lib_id "power:GND") (at 242.57 21.59 0) (unit 1)
     (in_bom yes) (on_board yes) (fields_autoplaced)
@@
     )
     (property "Datasheet" "" (id 3) (at 267.97 46.99 0)
+      (effects (font (size 1.27 1.27)) hide)
+    )
+    (pin "1")
+  )
+  (symbol (lib_id "power:GND") (at 59.69 193.04 0) (unit 1)
+    (in_bom yes) (on_board yes) (fields_autoplaced)
+    (property "Reference" "#PWR02" (id 0) (at 59.69 199.39 0)
+      (effects (font (size 1.27 1.27)) hide)
+    )
+    (property "Value" "GND" (id 1) (at 59.69 198.12 0)
+      (effects (font (size 1.27 1.27)) hide)
+    )
+    (property "Footprint" "" (id 2) (at 59.69 193.04 0)
+      (effects (font (size 1.27 1.27)) hide)
+    )
+    (property "Datasheet" "" (id 3) (at 59.69 193.04 0)
       (effects (font (size 1.27 1.27)) hide)
     )
@@
       (reference "#PWR01") (unit 1) (value "GND") (footprint "")
     )
+    (path "/5f6b1080-20a3-4632-95ab-7b720d91eec0"
+      (reference "#PWR02") (unit 1) (value "GND") (footprint "")
+    )
     (path "/5d07cb7e-c8e3-4ee6-8941-4590fa1e9acf"
       (reference "#PWR03") (unit 1) (value "GND") (footprint "")
@@
       (reference "J11") (unit 1) (value "OutToRPi") (footprint "Connector_PinHeader_2.54mm:PinHeader_1x02_P2.54mm_Vertical")
     )
+    (path "/1d0ef5db-c335-4d55-88dd-66a03b46c698"
+      (reference "J12") (unit 1) (value "LEDConn_01x05") (footprint "Connector_PinHeader_2.54mm:PinHeader_1x05_P2.54mm_Vertical")
+    )
+    (path "/4d0bd211-4794-4141-8b4c-fc5ed36fe38a/2faa9641-2ece-4171-8790-3945bf54da23"
+      (reference "J13") (unit 1) (value "RPiConn_01x03") (footprint "Connector_PinSocket_2.54mm:PinSocket_1x03_P2.54mm_Vertical")
+    )
     (path "/ba21e8b0-efb7-4c13-98e2-ebc8a39461f9"

Commit message: Final changes to PCB after footprint tests.
Parts:
- J1: footprint Connector_BarrelJack:BarrelJack_CUI_PJ-102AH_Horizontal -> Connector_BarrelJack:BarrelJack_GCT_DCJ200-10-A_Horizontal
Changed lines of the file:
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@@
       (effects (font (size 1.27 1.27)) (justify left))
     )
-    (property "Footprint" "Connector_BarrelJack:BarrelJack_CUI_PJ-102AH_Horizontal" (id 2) (at 248.92 17.78 0)
+    (property "Footprint" "Connector_BarrelJack:BarrelJack_GCT_DCJ200-10-A_Horizontal" (id 2) (at 248.92 17.78 0)
       (effects (font (size 1.27 1.27)) hide)
     )
@@
     )
     (path "/3e1ccb16-5496-4985-9aa9-d268c89cac5f"
-      (reference "J1") (unit 1) (value "BarrelJack") (footprint "Connector_BarrelJack:BarrelJack_CUI_PJ-102AH_Horizontal")
+      (reference "J1") (unit 1) (value "BarrelJack") (footprint "Connector_BarrelJack:BarrelJack_GCT_DCJ200-10-A_Horizontal")
     )
     (path "/9119ee79-ac43-4908-ba85-62b847bd6c6c"
